Commit message: Update Sensorintegration

File: config/ur10e_joint_limited_hand_conf.urdf.xacro (robot description, xacro)
@@ -51,5 +51,5 @@
             </geometry>
         </collision>
-<inertial>
+        <inertial>
             <mass value="7.778" />
             <origin rpy="0 0 0" xyz="0.0 0.0 0.0" />
@@ -398,5 +398,6 @@
         <axis xyz="0 1 0" />
         <limit effort="20" lower="0.00" upper="0.04" velocity="0.1" />
-        <dynamics damping="5.0" friction="0.02" />
+        <dynamics damping="5.0" friction="0.01" />
+        <!--dynamics damping="5.0" friction="0.02" /-->
     </joint>
     <joint name="panda_finger_joint2" type="prismatic">
@@ -407,5 +408,6 @@
         <limit effort="20" lower="0.00" upper="0.04" velocity="0.2" />
         <mimic joint="panda_finger_joint1" />
-        <dynamics damping="5.0" friction="0.02" />
+        <dynamics damping="5.0" friction="0.01" />
+        <!--dynamics damping="5.0" friction="0.02" /-->
     </joint>
     <joint name="$tool0-panda_hand" type="fixed">
